Commit message: update

File: install/small_arm_description/share/small_arm_description/urdf/small_arm.ros2_control.xacro (robot description, xacro)
@@ -7,5 +7,5 @@
         <param name="usb_port">/dev/ttyUSB0</param>
         <param name="baud_rate">115200</param>
-        <param name="use_dummy">false</param>
+        <param name="use_dummy">true</param>
       </hardware>
       <joint name="joint1">
@@ -57,5 +57,5 @@
         <state_interface name="effort"/>
       </joint>
-      <joint name="joint7">
+      <joint name="gripper_joint1">
         <param name="id">7</param>
         <command_interface name="position"/>
@@ -65,4 +65,16 @@
         <state_interface name="effort"/>
       </joint>
+      <!-- <hardware>
+          <plugin>fake_components/GenericSystem</plugin>
+      </hardware>
+      <joint name="gripper_joint2">
+        <param name="mimic">gripper_joint1</param>
+        <param name="multiplier">-1</param>
+        <command_interface name="position"/>
+        <command_interface name="velocity"/>
+        <state_interface name="position"/>
+        <state_interface name="velocity"/>
+        <state_interface name="effort"/>
+      </joint> -->
     </ros2_control>
   </xacro:macro>

File: install/small_arm_description/share/small_arm_description/urdf/small_arm.xacro (robot description, xacro)
@@ -12,19 +12,19 @@
   </joint>
   <link name="${base_name}">
-    <inertial>
-      <origin xyz="-0.0002999964758485541 -0.01002821324623266 0.02805569132780727" rpy="0 0 0"/>
-      <mass value="1.29137439344346"/>
-      <inertia ixx="0.001017" iyy="0.000798" izz="0.00122" ixy="-0.0" iyz="-3.2e-05" ixz="0.0"/>
-    </inertial>
-    <visual>
-      <origin xyz="0 0 0" rpy="0 0 0"/>
-      <geometry>
+  <inertial>
+    <origin xyz="6.583680213469905e-06 -0.010020414765013672 0.028054295745135273" rpy="0 0 0"/>
+    <mass value="1.291881447401789"/>
+    <inertia ixx="0.001017" iyy="0.000798" izz="0.00122" ixy="-0.0" iyz="-3.2e-05" ixz="0.0"/>
+  </inertial>
+  <visual>
+    <origin xyz="0 0 0" rpy="0 0 0"/>
+    <geometry>
         <mesh filename="package://small_arm_description/meshes/base_link.stl" scale="0.001 0.001 0.001"/>
-      </geometry>
-      <material name="silver"/>
-    </visual>
-    <collision>
-      <origin xyz="0 0 0" rpy="0 0 0"/>
-      <geometry>
+    </geometry>
+    <material name="silver"/>
+  </visual>
+  <collision>
+    <origin xyz="0 0 0" rpy="0 0 0"/>
+    <geometry>
         <mesh filename="package://small_arm_description/meshes/base_link.stl" scale="0.001 0.001 0.001"/>
       </geometry>
@@ -32,19 +32,19 @@
   </link>
   <link name="link1">
-    <inertial>
-      <origin xyz="0.0005539067623238434 -2.1382866212631147e-05 0.03707065153568121" rpy="0 0 0"/>
-      <mass value="0.8171892676957183"/>
-      <inertia ixx="0.000382" iyy="0.000408" izz="0.00022" ixy="0.0" iyz="0.0" ixz="-3e-06"/>
-    </inertial>
-    <visual>
-      <origin xyz="0.0003 -4.1e-05 -0.053" rpy="0 0 0"/>
-      <geometry>
+  <inertial>
+    <origin xyz="0.0005537302728879505 -3.989448908630728e-05 0.037038629210684425" rpy="0 0 0"/>
+    <mass value="0.817449728930332"/>
+    <inertia ixx="0.000383" iyy="0.000409" izz="0.00022" ixy="0.0" iyz="0.0" ixz="-3e-06"/>
+  </inertial>
+  <visual>
+    <origin xyz="0.0 -4.1e-05 -0.053" rpy="0 0 0"/>
+    <geometry>
         <mesh filename="package://small_arm_description/meshes/link_1_1.stl" scale="0.001 0.001 0.001"/>
-      </geometry>
-      <material name="silver"/>
-    </visual>
-    <collision>
-      <origin xyz="0.0003 -4.1e-05 -0.053" rpy="0 0 0"/>
-      <geometry>
+    </geometry>
+    <material name="silver"/>
+  </visual>
+  <collision>
+    <origin xyz="0.0 -4.1e-05 -0.053" rpy="0 0 0"/>
+    <geometry>
         <mesh filename="package://small_arm_description/meshes/link_1_1.stl" scale="0.001 0.001 0.001"/>
       </geometry>
@@ -52,19 +52,19 @@
   </link>
   <link name="link2">
-    <inertial>
-      <origin xyz="-0.024402873741152922 -0.0009180927250929553 0.08726652583609527" rpy="0 0 0"/>
-      <mass value="2.211704028669612"/>
-      <inertia ixx="0.005529" iyy="0.005935" izz="0.001201" ixy="-0.0" iyz="8.6e-05" ixz="-2.5e-05"/>
-    </inertial>
-    <visual>
-      <origin xyz="-0.0242 0.0 -0.109" rpy="0 0 0"/>
-      <geometry>
+  <inertial>
+    <origin xyz="-0.024427682432744808 -0.0006951262423943992 0.09244818830678549" rpy="0 0 0"/>
+    <mass value="2.530467328750089"/>
+    <inertia ixx="0.007365" iyy="0.007836" izz="0.001385" ixy="-0.0" iyz="0.00013" ixz="-3e-05"/>
+  </inertial>
+  <visual>
+    <origin xyz="-0.0245 0.0 -0.109" rpy="0 0 0"/>
+    <geometry>
         <mesh filename="package://small_arm_description/meshes/link_2_1.stl" scale="0.001 0.001 0.001"/>
-      </geometry>
-      <material name="silver"/>
-    </visual>
-    <collision>
-      <origin xyz="-0.0242 0.0 -0.109" rpy="0 0 0"/>
-      <geometry>
+    </geometry>
+    <material name="silver"/>
+  </visual>
+  <collision>
+    <origin xyz="-0.0245 0.0 -0.109" rpy="0 0 0"/>
+    <geometry>
         <mesh filename="package://small_arm_description/meshes/link_2_1.stl" scale="0.001 0.001 0.001"/>
       </geometry>
@@ -72,19 +72,19 @@
   </link>
   <link name="link3">
-    <inertial>
-      <origin xyz="-0.024562745448922518 0.06329760185292234 0.004043498969020454" rpy="0 0 0"/>
-      <mass value="1.4560374497113304"/>
-      <inertia ixx="0.001645" iyy="0.001003" izz="0.001935" ixy="2e-06" iyz="-1.2e-05" ixz="-0.0"/>
-    </inertial>
-    <visual>
-      <origin xyz="-0.0241 -0.0 -0.264" rpy="0 0 0"/>
-      <geometry>
+  <inertial>
+    <origin xyz="-0.02460425910708876 0.07785646945010617 0.0036503427791832466" rpy="0 0 0"/>
+    <mass value="1.5891656965493803"/>
+    <inertia ixx="0.002408" iyy="0.001132" izz="0.002797" ixy="3e-06" iyz="-5.1e-05" ixz="0.0"/>
+  </inertial>
+  <visual>
+    <origin xyz="-0.0244 -0.0 -0.279" rpy="0 0 0"/>
+    <geometry>
         <mesh filename="package://small_arm_description/meshes/link_3_1.stl" scale="0.001 0.001 0.001"/>
-      </geometry>
-      <material name="silver"/>
-    </visual>
-    <collision>
-      <origin xyz="-0.0241 -0.0 -0.264" rpy="0 0 0"/>
-      <geometry>
+    </geometry>
+    <material name="silver"/>
+  </visual>
+  <collision>
+    <origin xyz="-0.0244 -0.0 -0.279" rpy="0 0 0"/>
+    <geometry>
         <mesh filename="package://small_arm_description/meshes/link_3_1.stl" scale="0.001 0.001 0.001"/>
       </geometry>
@@ -92,19 +92,19 @@
   </link>
   <link name="link4">
-    <inertial>
-      <origin xyz="-0.0001915907936059267 0.028749765366266278 1.3933167071766839e-05" rpy="0 0 0"/>
-      <mass value="0.4445934457308041"/>
-      <inertia ixx="0.000143" iyy="8.2e-05" izz="0.00014" ixy="1e-06" iyz="-0.0" ixz="-0.0"/>
-    </inertial>
-    <visual>
-      <origin xyz="0.0006 -0.100766 -0.265316" rpy="0 0 0"/>
-      <geometry>
+  <inertial>
+    <origin xyz="0.0005678122855020656 0.028502036892318075 0.00010812835093654272" rpy="0 0 0"/>
+    <mass value="0.4500719035752892"/>
+    <inertia ixx="0.000146" iyy="8.3e-05" izz="0.000143" ixy="-1e-06" iyz="-0.0" ixz="-0.0"/>
+  </inertial>
+  <visual>
+    <origin xyz="0.0003 -0.121766 -0.280316" rpy="0 0 0"/>
+    <geometry>
         <mesh filename="package://small_arm_description/meshes/link_4_1.stl" scale="0.001 0.001 0.001"/>
-      </geometry>
-      <material name="silver"/>
-    </visual>
-    <collision>
-      <origin xyz="0.0006 -0.100766 -0.265316" rpy="0 0 0"/>
-      <geometry>
+    </geometry>
+    <material name="silver"/>
+  </visual>
+  <collision>
+    <origin xyz="0.0003 -0.121766 -0.280316" rpy="0 0 0"/>
+    <geometry>
         <mesh filename="package://small_arm_description/meshes/link_4_1.stl" scale="0.001 0.001 0.001"/>
       </geometry>
@@ -112,19 +112,19 @@
   </link>
   <link name="link5">
-    <inertial>
-      <origin xyz="-0.019004907946417172 0.007238676029536678 -0.043336314243680424" rpy="0 0 0"/>
-      <mass value="0.970501435691462"/>
-      <inertia ixx="0.00064" iyy="0.000557" izz="0.000514" ixy="-1e-06" iyz="-1.4e-05" ixz="-0.0"/>
-    </inertial>
-    <visual>
-      <origin xyz="-0.0174 -0.144647 -0.265316" rpy="0 0 0"/>
-      <geometry>
+  <inertial>
+    <origin xyz="-0.019068054583883113 0.009694576419165046 -0.04274059819483081" rpy="0 0 0"/>
+    <mass value="1.0859764685043407"/>
+    <inertia ixx="0.000829" iyy="0.00064" izz="0.000658" ixy="-0.0" iyz="-0.0001" ixz="-0.0"/>
+  </inertial>
+  <visual>
+    <origin xyz="-0.0187 -0.165647 -0.280441" rpy="0 0 0"/>
+    <geometry>
         <mesh filename="package://small_arm_description/meshes/link_5_1.stl" scale="0.001 0.001 0.001"/>
-      </geometry>
-      <material name="silver"/>
-    </visual>
-    <collision>
-      <origin xyz="-0.0174 -0.144647 -0.265316" rpy="0 0 0"/>
-      <geometry>
+    </geometry>
+    <material name="silver"/>
+  </visual>
+  <collision>
+    <origin xyz="-0.0187 -0.165647 -0.280441" rpy="0 0 0"/>
+    <geometry>
         <mesh filename="package://small_arm_description/meshes/link_5_1.stl" scale="0.001 0.001 0.001"/>
       </geometry>
@@ -132,40 +132,40 @@
   </link>
   <link name="link6">
-    <inertial>
-      <origin xyz="-5.506012312750386e-15 4.949917709884399e-07 -0.0026212148467256724" rpy="0 0 0"/>
-      <mass value="0.025512046719187297"/>
-      <inertia ixx="2e-06" iyy="2e-06" izz="4e-06" ixy="0.0" iyz="0.0" ixz="-0.0"/>
-    </inertial>
-    <visual>
-      <origin xyz="0.0016 -0.144647 -0.196297" rpy="0 0 0"/>
-      <geometry>
-        <mesh filename="package://small_arm_description/meshes/link_6_1.stl" scale="0.001 0.001 0.001"/>
-      </geometry>
-      <material name="silver"/>
-    </visual>
-    <collision>
-      <origin xyz="0.0016 -0.144647 -0.196297" rpy="0 0 0"/>
-      <geometry>
-        <mesh filename="package://small_arm_description/meshes/link_6_1.stl" scale="0.001 0.001 0.001"/>
+  <inertial>
+    <origin xyz="0.004492294331015427 0.0003709408309400253 -0.019015271355907637" rpy="0 0 0"/>
+    <mass value="0.5127274279729177"/>
+    <inertia ixx="9.5e-05" iyy="0.000226" izz="0.000235" ixy="-1e-06" iyz="0.0" ixz="1e-06"/>
+  </inertial>
+  <visual>
+    <origin xyz="0.0004 -0.165647 -0.205922" rpy="0 0 0"/>
+    <geometry>
+        <mesh filename="package://small_arm_description/meshes/Claw_base_1.stl" scale="0.001 0.001 0.001"/>
+    </geometry>
+    <material name="silver"/>
+  </visual>
+  <collision>
+    <origin xyz="0.0004 -0.165647 -0.205922" rpy="0 0 0"/>
+    <geometry>
+        <mesh filename="package://small_arm_description/meshes/Claw_base_1.stl" scale="0.001 0.001 0.001"/>
       </geometry>
     </collision>
   </link>
   <link name="gripper_link1">
-    <inertial>
-      <origin xyz="0.009922614801186412 -0.01909950500842314 -0.024668286066997724" rpy="0 0 0"/>
-      <mass value="0.16533614239781452"/>
-      <inertia ixx="0.000142" iyy="7.7e-05" izz="8.2e-05" ixy="-0.0" iyz="-0.0" ixz="5e-06"/>
-    </inertial>
-    <visual>
-      <origin xyz="-0.0204 -0.163647 -0.169647" rpy="0 0 0"/>
-      <geometry>
-        <mesh filename="package://small_arm_description/meshes/Craw_2_1.stl" scale="0.001 0.001 0.001"/>
-      </geometry>
-      <material name="silver"/>
-    </visual>
-    <collision>
-      <origin xyz="-0.0204 -0.163647 -0.169647" rpy="0 0 0"/>
-      <geometry>
-        <mesh filename="package://small_arm_description/meshes/Craw_2_1.stl" scale="0.001 0.001 0.001"/>
+  <inertial>
+    <origin xyz="0.009553177578958301 -0.019099491341480757 -0.027462032562735744" rpy="0 0 0"/>
+    <mass value="0.3481919018430052"/>
+    <inertia ixx="0.000338" iyy="0.000245" izz="0.000155" ixy="0.0" iyz="-0.0" ixz="2.6e-05"/>
+  </inertial>
+  <visual>
+    <origin xyz="-0.0216 -0.184647 -0.184772" rpy="0 0 0"/>
+    <geometry>
+        <mesh filename="package://small_arm_description/meshes/Claw_1_1.stl" scale="0.001 0.001 0.001"/>
+    </geometry>
+    <material name="silver"/>
+  </visual>
+  <collision>
+    <origin xyz="-0.0216 -0.184647 -0.184772" rpy="0 0 0"/>
+    <geometry>
+        <mesh filename="package://small_arm_description/meshes/Claw_1_1.stl" scale="0.001 0.001 0.001"/>
       </geometry>
     </collision>
@@ -173,44 +173,44 @@
 <link name="gripper_link2">
   <inertial>
-    <origin xyz="-0.004639846314339198 0.0002472053469017299 -0.02547670727420101" rpy="0 0 0"/>
-    <mass value="0.6910133017831432"/>
-    <inertia ixx="0.000328" iyy="0.000563" izz="0.000489" ixy="-3e-06" iyz="-1e-06" ixz="-0.000126"/>
-  </inertial>
-  <visual>
-    <origin xyz="0.0016 -0.144647 -0.190797" rpy="0 0 0"/>
-    <geometry>
-      <mesh filename="package://small_arm_description/meshes/Craw_1_1.stl" scale="0.001 0.001 0.001"/>
-    </geometry>
-    <material name="silver"/>
-  </visual>
-  <collision>
-    <origin xyz="0.0016 -0.144647 -0.190797" rpy="0 0 0"/>
-    <geometry>
-      <mesh filename="package://small_arm_description/meshes/Craw_1_1.stl" scale="0.001 0.001 0.001"/>
-    </geometry>
-  </collision>
-</link>
+    <origin xyz="-0.008862773747378604 -0.01908264305352636 -0.025794573876087107" rpy="0 0 0"/>
+    <mass value="0.3632084794432327"/>
+    <inertia ixx="0.000361" iyy="0.000263" izz="0.000164" ixy="0.0" iyz="0.0" ixz="-3.1e-05"/>
+  </inertial>
+  <visual>
+    <origin xyz="0.0224 -0.184582 -0.184772" rpy="0 0 0"/>
+    <geometry>
+        <mesh filename="package://small_arm_description/meshes/Claw_2_1.stl" scale="0.001 0.001 0.001"/>
+    </geometry>
+    <material name="silver"/>
+  </visual>
+  <collision>
+    <origin xyz="0.0224 -0.184582 -0.184772" rpy="0 0 0"/>
+    <geometry>
+        <mesh filename="package://small_arm_description/meshes/Claw_2_1.stl" scale="0.001 0.001 0.001"/>
+      </geometry>
+    </collision>
+  </link>
   <link name="camera_link">
-    <inertial>
-      <origin xyz="-0.02250186173818042 -4.850013210841442e-05 -0.012169837419761076" rpy="0 0 0"/>
-      <mass value="0.3783798760930688"/>
-      <inertia ixx="3.5e-05" iyy="0.00024" izz="0.000238" ixy="-0.0" iyz="-0.0" ixz="0.0"/>
-    </inertial>
-    <visual>
-      <origin xyz="-0.0209 -0.194439 -0.219247" rpy="0 0 0"/>
-      <geometry>
-        <mesh filename="package://small_arm_description/meshes/RealSence_1.stl" scale="0.001 0.001 0.001"/>
-      </geometry>
-      <material name="silver"/>
-    </visual>
-    <collision>
-      <origin xyz="-0.0209 -0.194439 -0.219247" rpy="0 0 0"/>
-      <geometry>
-        <mesh filename="package://small_arm_description/meshes/RealSence_1.stl" scale="0.001 0.001 0.001"/>
+  <inertial>
+    <origin xyz="-0.022501861739521612 -4.8500070798096484e-05 -0.012169837448304244" rpy="0 0 0"/>
+    <mass value="0.37837987609307205"/>
+    <inertia ixx="3.5e-05" iyy="0.00024" izz="0.000238" ixy="-0.0" iyz="-0.0" ixz="0.0"/>
+  </inertial>
+  <visual>
+    <origin xyz="-0.0222 -0.225439 -0.254372" rpy="0 0 0"/>
+    <geometry>
+        <mesh filename="package://small_arm_description/meshes/Camera_1.stl" scale="0.001 0.001 0.001"/>
+    </geometry>
+    <material name="silver"/>
+  </visual>
+  <collision>
+    <origin xyz="-0.0222 -0.225439 -0.254372" rpy="0 0 0"/>
+    <geometry>
+        <mesh filename="package://small_arm_description/meshes/Camera_1.stl" scale="0.001 0.001 0.001"/>
       </geometry>
     </collision>
   </link>
   <joint name="joint1" type="revolute">
-    <origin xyz="-0.0003 4.1e-05 0.053" rpy="0 0 0"/>
+    <origin xyz="0.0 4.1e-05 0.053" rpy="0 0 0"/>
     <parent link="${base_name}"/>
     <child link="link1"/>
@@ -234,5 +234,5 @@
   </joint>
   <joint name="joint3" type="revolute">
-    <origin xyz="-0.0001 0.0 0.155" rpy="0 0 0"/>
+    <origin xyz="-0.0001 0.0 0.17" rpy="0 0 0"/>
     <parent link="link2"/>
     <child link="link3"/>
@@ -245,8 +245,8 @@
   </joint>
   <joint name="joint4" type="revolute">
-    <origin xyz="-0.0247 0.100766 0.001316" rpy="0 0 0"/>
+    <origin xyz="-0.0247 0.121766 0.001316" rpy="0 0 0"/>
     <parent link="link3"/>
     <child link="link4"/>
-    <axis xyz="-0.0 -1.0 -0.0"/>
+    <axis xyz="-0.0 1.0 -0.0"/>
     <limit
       lower="-3.14"
@@ -256,5 +256,5 @@
   </joint>
   <joint name="joint5" type="revolute">
-    <origin xyz="0.018 0.043881 0.0" rpy="0 0 0"/>
+    <origin xyz="0.019 0.043881 0.000125" rpy="0 0 0"/>
     <parent link="link4"/>
     <child link="link5"/>
@@ -267,5 +267,5 @@
   </joint>
   <joint name="joint6" type="revolute">
-    <origin xyz="-0.019 0.0 -0.069019" rpy="0 0 0"/>
+    <origin xyz="-0.0191 0.0 -0.074519" rpy="0 0 0"/>
     <parent link="link5"/>
     <child link="link6"/>
@@ -277,7 +277,7 @@
       velocity="4.8" />
   </joint>
-  <joint name="joint7" type="revolute">
+  <joint name="gripper_joint1" type="revolute">
     <origin xyz="0.022 0.019 -0.02115" rpy="0 0 0"/>
-    <parent link="gripper_link2"/>
+    <parent link="link6"/>
     <child link="gripper_link1"/>
     <axis xyz="0.0 1.0 0.0"/>
@@ -288,11 +288,23 @@
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
File: install/small_arm_moveit_config/share/small_arm_moveit_config/config/small_arm.ros2_control.xacro (robot description, xacro)
@@ -12,5 +12,5 @@
                     <param name="usb_port">/dev/ttyUSB0</param>
                     <param name="baud_rate">115200</param>
-                    <param name="use_dummy">true</param>
+                    <param name="use_dummy">false</param>
                 </xacro:if>
             </hardware>
@@ -63,5 +63,5 @@
         <state_interface name="effort"/>
       </joint>
-      <joint name="joint7">
+      <joint name="gripper_joint1">
         <param name="id">7</param>
         <command_interface name="position"/>
@@ -71,57 +71,10 @@
         <state_interface name="effort"/>
       </joint>
-            <!-- <joint name="joint1">
-            <param name="id">1</param>
+            <!-- <joint name="gripper_joint2">
+                <param name="mimic">gripper_joint1</param>
+                <param name="multiplier">-1</param>
                 <command_interface name="position"/>
                 <state_interface name="position">
-                  <param name="initial_value">${initial_positions['joint1']}</param>
-                </state_interface>
-                <state_interface name="velocity"/>
-            </joint>
-            <joint name="joint2">
-            <param name="id">2</param>
-                <command_interface name="position"/>
-                <state_interface name="position">
-                  <param name="initial_value">${initial_positions['joint2']}</param>
-                </state_interface>
-                <state_interface name="velocity"/>
-            </joint>
-            <joint name="joint3">
-            <param name="id">3</param>
-                <command_interface name="position"/>
-                <state_interface name="position">
-                  <param name="initial_value">${initial_positions['joint3']}</param>
-                </state_interface>
-                <state_interface name="velocity"/>
-            </joint>
-            <joint name="joint4">
-            <param name="id">4</param>
-                <command_interface name="position"/>
-                <state_interface name="position">
-                  <param name="initial_value">${initial_positions['joint4']}</param>
-                </state_interface>
-                <state_interface name="velocity"/>
-            </joint>
-            <joint name="joint5">
-            <param name="id">5</param>
-                <command_interface name="position"/>
-                <state_interface name="position">
-                  <param name="initial_value">${initial_positions['joint5']}</param>
-                </state_interface>
-                <state_interface name="velocity"/>
-            </joint>
-            <joint name="joint6">
-            <param name="id">6</param>
-                <command_interface name="position"/>
-                <state_interface name="position">
-                  <param name="initial_value">${initial_positions['joint6']}</param>
-                </state_interface>
-                <state_interface name="velocity"/>
-            </joint>
-            <joint name="joint7">
-            <param name="id">7</param>
-                <command_interface name="position"/>
-                <state_interface name="position">
-                  <param name="initial_value">${initial_positions['joint7']}</param>
+                  <param name="initial_value">${initial_positions['gripper_joint1']}</param>
                 </state_interface>
                 <state_interface name="velocity"/>

File: install/small_arm_moveit_config/share/small_arm_moveit_config/config/small_arm.urdf.xacro (robot description, xacro)
@@ -2,5 +2,5 @@
 <robot xmlns:xacro="http://www.ros.org/wiki/xacro" name="small_arm">
     <xacro:arg name="initial_positions_file" default="initial_positions.yaml" />
-    <xacro:arg name="ros2_control_hardware_type" default="mock_components" />
+    <xacro:arg name="ros2_control_hardware_type" default="fake" />
     <!-- Import small_arm urdf file -->
     <xacro:include filename="$(find small_arm_description)/urdf/small_arm.urdf.xacro" />
